File: KiCAD-PCB/Shield Arduino.kicad_sch (KiCad schematic)
At the start: 23 parts, among them J1 Power, J2 Digital/PWM, J3 Analog, J4 Digital/PWM, U1 LTC1050CN8, U2 MCP41010

Commit message: Add files via upload
Connections:
- net +5V: no longer U2.5 (PA0)
- net GND: now also U2.5 (PA0), U2.6 (PW0); no longer U2.7 (PB0)
- net R2: now also U2.7 (PB0); no longer U2.6 (PW0)
Changed lines of the file:
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@@
   (junction (at 175.26 128.27) (diameter 0) (color 0 0 0 0)
   )
+  (junction (at 161.29 175.26) (diameter 0) (color 0 0 0 0)
+  )
   (junction (at 243.84 41.91) (diameter 0) (color 0 0 0 0)
   )
@@
   (junction (at 224.79 39.37) (diameter 0) (color 0 0 0 0)
   )
-  (junction (at 151.13 189.23) (diameter 0) (color 0 0 0 0)
-  )
   (junction (at 165.1 134.62) (diameter 0) (color 0 0 0 0)
   )
@@
   )
   (junction (at 224.79 59.69) (diameter 0) (color 0 0 0 0)
-  )
-  (junction (at 151.13 166.37) (diameter 0) (color 0 0 0 0)
   )
   (junction (at 46.99 21.59) (diameter 0) (color 0 0 0 0)
@@
     (stroke (width 0) (type default))
   )
-  (wire (pts (xy 151.13 189.23) (xy 151.13 190.5))
+  (wire (pts (xy 151.13 187.96) (xy 151.13 190.5))
+    (stroke (width 0) (type default))
+  )
+  (wire (pts (xy 161.29 175.26) (xy 161.29 177.8))
     (stroke (width 0) (type default))
   )
@@
     (stroke (width 0) (type default))
   )
-  (wire (pts (xy 151.13 187.96) (xy 151.13 189.23))
-    (stroke (width 0) (type default))
-  )
   (wire (pts (xy 224.79 39.37) (xy 229.87 39.37))
     (stroke (width 0) (type default))
@@
     (stroke (width 0) (type solid))
   )
-  (wire (pts (xy 151.13 163.83) (xy 151.13 166.37))
-    (stroke (width 0) (type default))
-  )
   (wire (pts (xy 139.7 73.66) (xy 138.43 73.66))
     (stroke (width 0) (type default))
@@
     (stroke (width 0) (type default))
   )
-  (wire (pts (xy 161.29 166.37) (xy 151.13 166.37))
-    (stroke (width 0) (type default))
-  )
   (wire (pts (xy 224.79 59.69) (xy 270.51 59.69))
     (stroke (width 0) (type default))
@@
     (stroke (width 0) (type default))
   )
-  (wire (pts (xy 161.29 175.26) (xy 161.29 166.37))
-    (stroke (width 0) (type default))
-  )
   (wire (pts (xy 142.24 134.62) (xy 142.24 139.7))
     (stroke (width 0) (type default))
@@
     (stroke (width 0) (type default))
   )
+  (wire (pts (xy 161.29 175.26) (xy 162.56 175.26))
+    (stroke (width 0) (type default))
+  )
   (wire (pts (xy 140.97 49.53) (xy 140.97 46.99))
     (stroke (width 0) (type default))
@@
     (stroke (width 0) (type default))
   )
-  (wire (pts (xy 161.29 189.23) (xy 151.13 189.23))
-    (stroke (width 0) (type default))
-  )
   (wire (pts (xy 175.26 128.27) (xy 176.53 128.27))
     (stroke (width 0) (type default))
@@
     (stroke (width 0) (type default))
   )
-  (wire (pts (xy 151.13 166.37) (xy 151.13 167.64))
-    (stroke (width 0) (type default))
-  )
-  (wire (pts (xy 161.29 180.34) (xy 161.29 189.23))
+  (wire (pts (xy 151.13 163.83) (xy 151.13 167.64))
     (stroke (width 0) (type default))
   )
@@
     )
   )
-  (global_label "R2" (shape input) (at 161.29 177.8 0) (fields_autoplaced)
-    (effects (font (size 1.27 1.27)) (justify left))
-    (property "Intersheetrefs" "${INTERSHEET_REFS}" (at 166.7704 177.8 0)
+  (global_label "R2" (shape input) (at 161.29 180.34 0) (fields_autoplaced)
+    (effects (font (size 1.27 1.27)) (justify left))
+    (property "Intersheetrefs" "${INTERSHEET_REFS}" (at 166.7704 180.34 0)
       (effects (font (size 1.27 1.27)) (justify left) hide)
     )
@@
         )
       )
+    )
+  )
+  (symbol (lib_id "power:GND") (at 162.56 175.26 90) (unit 1)
+    (in_bom yes) (on_board yes) (dnp no)
+    (property "Reference" "#PWR017" (at 168.91 175.26 0)
+      (effects (font (size 1.27 1.27)) hide)
+    )
+    (property "Value" "GND" (at 166.37 175.26 0)
+      (effects (font (size 1.27 1.27)))
+    )
+    (property "Footprint" "" (at 162.56 175.26 0)
+      (effects (font (size 1.27 1.27)))
+    )
+    (property "Datasheet" "" (at 162.56 175.26 0)
+      (effects (font (size 1.27 1.27)))
+    )
+    (pin "1")
+    (instances
+      (project "Shield Arduino"
+        (path "/e63e39d7-6ac0-4ffd-8aa3-1841a4541b55"
+          (reference "#PWR017") (unit 1)
+        )
+      )
