File: KiCAD-PCB/Shield Arduino.kicad_pcb (KiCad board)
At the start: 2 copper layers, 71.1 x 58.4 mm, 27 parts, among them J1 Power, J2 Digital/PWM, J3 Analog, J4 Digital/PWM, U1 LTC1050CN8, U2 MCP41010

Commit message: Add files via upload
Connections:
- U2 pad 5: +5V -> GND
- U2 pad 6: R2 -> GND
- U2 pad 7: GND -> R2
Routing:
- net +5V: track 206.3 -> 192.5 mm
- net D11: track 49.4 -> 42.4 mm
Changed lines of the file:
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@@
       (net 1 "GND") (pinfunction "VSS") (pintype "power_in"))
     (pad "5" thru_hole oval (at 7.62 7.62 270) (size 1.6 1.6) (drill 0.8) (layers "*.Cu" "*.Mask")
-      (net 3 "+5V") (pinfunction "PA0") (pintype "passive"))
+      (net 1 "GND") (pinfunction "PA0") (pintype "passive"))
     (pad "6" thru_hole oval (at 7.62 5.08 270) (size 1.6 1.6) (drill 0.8) (layers "*.Cu" "*.Mask")
-      (net 10 "R2") (pinfunction "PW0") (pintype "passive"))
+      (net 1 "GND") (pinfunction "PW0") (pintype "passive"))
     (pad "7" thru_hole oval (at 7.62 2.54 270) (size 1.6 1.6) (drill 0.8) (layers "*.Cu" "*.Mask")
-      (net 1 "GND") (pinfunction "PB0") (pintype "passive"))
+      (net 10 "R2") (pinfunction "PB0") (pintype "passive"))
     (pad "8" thru_hole oval (at 7.62 0 270) (size 1.6 1.6) (drill 0.8) (layers "*.Cu" "*.Mask")
       (net 3 "+5V") (pinfunction "VDD") (pintype "power_in"))
@@
   (segment (start 150.8 68.317919) (end 148.202081 65.72) (width 0.8) (layer "B.Cu") (net 3))
   (segment (start 143.18 59.36) (end 143.18 61.9) (width 0.8) (layer "B.Cu") (net 3))
-  (segment (start 125.4 61.9) (end 120.32 61.9) (width 0.8) (layer "B.Cu") (net 3))
-  (segment (start 126.66 63.16) (end 125.4 61.9) (width 0.8) (layer "B.Cu") (net 3))
   (segment (start 158.42 64.44) (end 158.42 59.36) (width 0.8) (layer "B.Cu") (net 3))
   (segment (start 135.56 65.72) (end 126.66 65.72) (width 0.8) (layer "B.Cu") (net 3))
-  (segment (start 119.04 63.18) (end 119.04 65.72) (width 0.8) (layer "B.Cu") (net 3))
   (segment (start 148.202081 65.72) (end 135.56 65.72) (width 0.8) (layer "B.Cu") (net 3))
   (segment (start 108.88 80.96) (end 107.62 82.22) (width 0.8) (layer "B.Cu") (net 3))
@@
   (segment (start 168.58 91.042081) (end 166.04 88.502081) (width 0.8) (layer "B.Cu") (net 3))
   (segment (start 143.18 61.9) (end 139.36 65.72) (width 0.8) (layer "B.Cu") (net 3))
-  (segment (start 126.66 65.72) (end 126.66 63.16) (width 0.8) (layer "B.Cu") (net 3))
   (segment (start 168.58 97.46) (end 168.58 91.042081) (width 0.8) (layer "B.Cu") (net 3))
   (segment (start 139.36 65.72) (end 135.56 65.72) (width 0.8) (layer "B.Cu") (net 3))
@@
   (segment (start 112.7 100) (end 107.62 94.92) (width 0.8) (layer "B.Cu") (net 3))
   (segment (start 143.18 55.617919) (end 147.057919 51.74) (width 0.8) (layer "B.Cu") (net 3))
-  (segment (start 120.32 61.9) (end 119.04 63.18) (width 0.8) (layer "B.Cu") (net 3))
   (segment (start 115.24 74.6) (end 117.78 74.6) (width 0.8) (layer "B.Cu") (net 5))
+  (segment (start 117.78 72.06) (end 115.24 74.6) (width 0.8) (layer "B.Cu") (net 5))
   (segment (start 110.14 74.6) (end 115.24 74.6) (width 0.8) (layer "B.Cu") (net 5))
+  (segment (start 130.48 74.6) (end 133.02 72.06) (width 0.8) (layer "B.Cu") (net 5))
   (segment (start 120.32 77.14) (end 117.78 74.6) (width 0.8) (layer "B.Cu") (net 5))
-  (segment (start 130.48 74.6) (end 133.02 72.06) (width 0.8) (layer "B.Cu") (net 5))
-  (segment (start 117.78 72.06) (end 115.24 74.6) (width 0.8) (layer "B.Cu") (net 5))
   (segment (start 117.78 74.6) (end 130.48 74.6) (width 0.8) (layer "B.Cu") (net 5))
   (segment (start 106.34 70.8) (end 110.14 74.6) (width 0.8) (layer "B.Cu") (net 5))
@@
   (segment (start 150.8 87.3) (end 150.8 97.46) (width 0.8) (layer "B.Cu") (net 6))
   (segment (start 145.8 79.68) (end 148.34 77.14) (width 0.8) (layer "B.Cu") (net 9))
+  (segment (start 115.24 79.68) (end 117.78 82.22) (width 0.8) (layer "B.Cu") (net 9))
   (segment (start 106.34 78.42) (end 107.74 77.02) (width 0.8) (layer "B.Cu") (net 9))
   (segment (start 133.02 77.14) (end 130.48 79.68) (width 0.8) (layer "B.Cu") (net 9))
   (segment (start 107.74 77.02) (end 112.58 77.02) (width 0.8) (layer "B.Cu") (net 9))
-  (segment (start 115.24 79.68) (end 117.78 82.22) (width 0.8) (layer "B.Cu") (net 9))
   (segment (start 115.24 79.68) (end 130.48 79.68) (width 0.8) (layer "B.Cu") (net 9))
   (segment (start 112.58 77.02) (end 115.24 79.68) (width 0.8) (layer "B.Cu") (net 9))
   (segment (start 130.48 79.68) (end 145.8 79.68) (width 0.8) (layer "B.Cu") (net 9))
-  (segment (start 121.58 65.72) (end 117.9 69.4) (width 0.8) (layer "B.Cu") (net 10))
+  (segment (start 135.44 69.4) (end 120.32 69.4) (width 0.8) (layer "B.Cu") (net 10))
   (segment (start 110.16 69.4) (end 110.16 69.52) (width 0.8) (layer "B.Cu") (net 10))
+  (segment (start 120.44 69.4) (end 120.32 69.4) (width 0.8) (layer "B.Cu") (net 10))
+  (segment (start 117.78 69.4) (end 110.16 69.4) (width 0.8) (layer "B.Cu") (net 10))
+  (segment (start 124.12 65.72) (end 120.44 69.4) (width 0.8) (layer "B.Cu") (net 10))
+  (segment (start 120.32 69.4) (end 117.78 69.4) (width 0.8) (layer "B.Cu") (net 10))
   (segment (start 143.18 77.14) (end 140.64 74.6) (width 0.8) (layer "B.Cu") (net 10))
-  (segment (start 117.78 69.4) (end 110.16 69.4) (width 0.8) (layer "B.Cu") (net 10))
-  (segment (start 117.9 69.4) (end 117.78 69.4) (width 0.8) (layer "B.Cu") (net 10))
-  (segment (start 135.44 69.4) (end 117.78 69.4) (width 0.8) (layer "B.Cu") (net 10))
   (segment (start 140.64 74.6) (end 135.44 69.4) (width 0.8) (layer "B.Cu") (net 10))
   (segment (start 110.16 69.52) (end 108.88 70.8) (width 0.8) (layer "B.Cu") (net 10))
@@
   (segment (start 128.956 53.264) (end 124.12 58.1) (width 0.8) (layer "B.Cu") (net 15))
   (segment (start 128.956 49.2) (end 128.956 53.264) (width 0.8) (layer "B.Cu") (net 15))
-  (segment (start 134.036 49.2) (end 131.496 46.66) (width 0.8) (layer "B.Cu") (net 16))
-  (segment (start 131.496 46.66) (end 110.16 46.66) (width 0.8) (layer "B.Cu") (net 16))
-  (segment (start 110.16 54.28) (end 120.32 54.28) (width 0.8) (layer "B.Cu") (net 16))
-  (segment (start 121.58 55.54) (end 121.58 58.1) (width 0.8) (layer "B.Cu") (net 16))
-  (segment (start 107.62 51.74) (end 110.16 54.28) (width 0.8) (layer "B.Cu") (net 16))
-  (segment (start 120.32 54.28) (end 121.58 55.54) (width 0.8) (layer "B.Cu") (net 16))
-  (segment (start 110.16 46.66) (end 107.62 49.2) (width 0.8) (layer "B.Cu") (net 16))
-  (segment (start 121.58 58.1) (end 121.311573 58.1) (width 0.8) (layer "B.Cu") (net 16))
-  (segment (start 107.62 49.2) (end 107.62 51.74) (width 0.8) (layer "B.Cu") (net 16))
+  (segment (start 110.16 49.488427) (end 112.988427 46.66) (width 0.8) (layer "B.Cu") (net 16))
+  (segment (start 131.496 46.66) (end 134.036 49.2) (width 0.8) (layer "B.Cu") (net 16))
+  (segment (start 121.58 58.1) (end 117.76 54.28) (width 0.8) (layer "B.Cu") (net 16))
+  (segment (start 117.76 54.28) (end 112.7 54.28) (width 0.8) (layer "B.Cu") (net 16))
+  (segment (start 112.7 54.28) (end 110.16 51.74) (width 0.8) (layer "B.Cu") (net 16))
+  (segment (start 110.16 51.74) (end 110.16 49.488427) (width 0.8) (layer "B.Cu") (net 16))
+  (segment (start 112.988427 46.66) (end 131.496 46.66) (width 0.8) (layer "B.Cu") (net 16))
   (segment (start 136.576 50.724) (end 129.2 58.1) (width 0.8) (layer "B.Cu") (net 17))
   (segment (start 136.576 49.2) (end 136.576 50.724) (width 0.8) (layer "B.Cu") (net 17))

Commit message: Add files via upload
Parts:
- moved C6 4.61 mm to (168.6, 70.8)
- moved C4 3.95 mm to (149.5, 80.9), turned to 90 degrees
- moved U2 3.60 mm to (124.1, 55.5)
- moved C2 2.54 mm to (133.1, 84.8)
- moved R2 2.54 mm to (143.2, 84.8)
- moved R6 2.54 mm to (117.8, 84.8)
- moved C5 1.82 mm to (164.8, 68.3)
Routing:
- net +5V: track 192.5 -> 174.9 mm
- net D2: track 30.7 -> 25.8 mm
- net D11: track 42.4 -> 37.8 mm
- net R2: track 57.2 -> 52.8 mm
- net A0: track 35.2 -> 31.1 mm
- net Net-(U1-OUT): track 51.9 -> 55.6 mm
- net Net-(U1-+IN): track 36.5 -> 34.7 mm
- net D10: track 14.5 -> 16.0 mm
- net D13: track 10.9 -> 12.4 mm
- net A1: track 22.4 -> 23.5 mm
- net D4: track 24.6 -> 23.8 mm
